Commit message: updated urdf with base_footprint_joint for slam

File: evobot_description/urdf/evobot.xacro (robot description, xacro)
@@ -2,6 +2,12 @@
 <robot name="evobot" xmlns:xacro="http://www.ros.org/wiki/xacro">
 <xacro:include filename="$(find evobot_description)/urdf/materials.xacro" />
-<xacro:include filename="$(find evobot_description)/urdf/evobot.trans" />
+<!-- <xacro:include filename="$(find evobot_description)/urdf/evobot.trans" /> -->
 <xacro:include filename="$(find evobot_description)/urdf/evobot.gazebo" />
+<link name="base_footprint"/>
+<joint name="base_footprint_joint" type="fixed">
+  <parent link="base_footprint"/>
+  <child link="base_link"/>
+  <origin xyz="0 0 0" rpy="0 0 0"/>
+</joint>
 <link name="base_link">
   <inertial>

Commit message: added map

File: evobot_description/urdf/evobot.xacro (robot description, xacro)
@@ -14,5 +14,6 @@
     <origin xyz="0.0 0.0 0.0" rpy="0 0 0"/>
     <mass value="15.11"/>
-    <inertia ixx="0.0" iyy="0.0" izz="0.0" ixy="0.0" iyz="0.0" ixz="0.0"/>
+    <!-- Approximate box inertia computed for a ~0.4 x 0.3 x 0.2 m base, mass=15.11 kg -->
+    <inertia ixx="0.164" iyy="0.252" izz="0.315" ixy="0.0" iyz="0.0" ixz="0.0"/>
   </inertial>
   <visual>
@@ -152,5 +153,5 @@
 <link name="lidar_1">
   <inertial>
-    <origin xyz="0 0 0 0 0 0"/>
+    <origin xyz="0 0 0" rpy="0 0 0"/>
     <mass value="0.05"/>
     <inertia ixx="1e-5" iyy="1e-5" izz="1e-5" ixy="0" ixz="0" iyz="0"/>

Commit message: added maps and navigation launch for evobot

File: evobot_description/urdf/evobot.xacro (robot description, xacro)
@@ -31,4 +31,12 @@
   </collision>
 </link>
+<!-- IMU link -->
+<link name="imu_link">
+  <inertial>
+    <origin xyz="0 0 0" rpy="0 0 0"/>
+    <mass value="0.01"/>
+    <inertia ixx="1e-6" iyy="1e-6" izz="1e-6" ixy="0" ixz="0" iyz="0"/>
+  </inertial>
+</link>
 <link name="r_wheel_1">
   <inertial>
@@ -211,3 +219,8 @@
   <child link="lidar_1"/>
 </joint>
+<joint name="imu_joint" type="fixed">
+  <parent link="base_link"/>
+  <child link="imu_link"/>
+  <origin xyz="0 0 0" rpy="0 0 0"/>
+</joint>
 </robot>
